File: hw/ikea-fornuftig/ikea-fornuftig.kicad_pcb (KiCad board)
At the start: 4 copper layers, 123.2 x 39.8 mm, 0 parts

Commit message: Update
Routing:
- net (no net): track 0.00 -> 87.4 mm, vias 0 -> 2
Changed lines of the file:
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@@
-(kicad_pcb (version 20211014) (generator pcbnew)
+(kicad_pcb (version 20221018) (generator pcbnew)
   (general
     (thickness 1.56)
@@
     (pcbplotparams
       (layerselection 0x00010fc_ffffffff)
+      (plot_on_all_layers_selection 0x0000000_00000000)
       (disableapertmacros false)
       (usegerberextensions false)
@@
       (usegerberadvancedattributes true)
       (creategerberjobfile true)
-      (svguseinch false)
+      (dashed_line_dash_ratio 12.000000)
+      (dashed_line_gap_ratio 3.000000)
       (svgprecision 6)
-      (excludeedgelayer true)
       (plotframeref false)
       (viasonmask false)
@@
   )
   (net 0 "")
-  (gr_circle (center 115.9 94.85) (end 117.9 94.85) (layer "B.Mask") (width 2) (fill none))
-  (gr_circle (center 175.3 70.05) (end 177.3 70.05) (layer "B.Mask") (width 2) (fill none))
-  (gr_circle (center 175.3 70.05) (end 177.3 70.05) (layer "F.Mask") (width 2) (fill none))
-  (gr_circle (center 115.9 94.85) (end 117.9 94.85) (layer "F.Mask") (width 2) (fill none))
-  (gr_circle (center 120.9 94.85) (end 122.05 94.85) (layer "Edge.Cuts") (width 0.1) (fill none))
-  (gr_line (start 183.3 82.45) (end 183.3 83.45) (layer "Edge.Cuts") (width 0.1))
-  (gr_line (start 75.1 59.9) (end 75.1 99.7) (layer "Edge.Cuts") (width 0.1))
-  (gr_line (start 183.3 82.4) (end 183.3 81.4) (layer "Edge.Cuts") (width 0.1))
-  (gr_line (start 173.3 98.1) (end 174.3 98.1) (layer "Edge.Cuts") (width 0.1))
-  (gr_line (start 110.1 59.9) (end 75.1 59.9) (layer "Edge.Cuts") (width 0.1))
-  (gr_line (start 183.3 82.4) (end 184.3 82.4) (layer "Edge.Cuts") (width 0.1))
-  (gr_line (start 135.1 82.75) (end 135.1 83.75) (layer "Edge.Cuts") (width 0.1))
-  (gr_circle (center 115.9 94.85) (end 117.85 94.85) (layer "Edge.Cuts") (width 0.1) (fill none))
-  (gr_line (start 173.3 98.1) (end 172.3 98.1) (layer "Edge.Cuts") (width 0.1))
-  (gr_circle (center 175.3 70.05) (end 177.25 70.05) (layer "Edge.Cuts") (width 0.1) (fill none))
-  (gr_circle (center 180.3 70.05) (end 181.45 70.05) (layer "Edge.Cuts") (width 0.1) (fill none))
-  (gr_line (start 173.3 98.1) (end 173.3 97.1) (layer "Edge.Cuts") (width 0.1))
-  (gr_rect (start 110.1 59.9) (end 198.3 99.7) (layer "Edge.Cuts") (width 0.1) (fill none))
-  (gr_line (start 135.1 82.7) (end 134.1 82.7) (layer "Edge.Cuts") (width 0.1))
-  (gr_line (start 135.1 82.7) (end 135.1 81.7) (layer "Edge.Cuts") (width 0.1))
-  (gr_line (start 135.1 82.7) (end 136.1 82.7) (layer "Edge.Cuts") (width 0.1))
-  (gr_line (start 110.1 99.7) (end 75.1 99.7) (layer "Edge.Cuts") (width 0.1))
-  (gr_line (start 183.3 82.4) (end 182.3 82.4) (layer "Edge.Cuts") (width 0.1))
+  (gr_circle (center 115.9 94.85) (end 117.9 94.85)
+    (stroke (width 2) (type solid)) (fill none) (layer "B.Mask"))
+  (gr_circle (center 175.3 70.05) (end 177.3 70.05)
+    (stroke (width 2) (type solid)) (fill none) (layer "B.Mask"))
+  (gr_circle (center 175.3 70.05) (end 177.3 70.05)
+    (stroke (width 2) (type solid)) (fill none) (layer "F.Mask"))
+  (gr_circle (center 115.9 94.85) (end 117.9 94.85)
+    (stroke (width 2) (type solid)) (fill none) (layer "F.Mask"))
+  (gr_circle (center 120.9 94.85) (end 122.05 94.85)
+    (stroke (width 0.1) (type solid)) (fill none) (layer "Edge.Cuts"))
+  (gr_line (start 183.3 82.45) (end 183.3 83.45)
+    (stroke (width 0.1) (type solid)) (layer "Edge.Cuts"))
+  (gr_line (start 75.1 59.9) (end 75.1 99.7)
+    (stroke (width 0.1) (type solid)) (layer "Edge.Cuts"))
+  (gr_line (start 183.3 82.4) (end 183.3 81.4)
+    (stroke (width 0.1) (type solid)) (layer "Edge.Cuts"))
+  (gr_line (start 173.3 98.1) (end 174.3 98.1)
+    (stroke (width 0.1) (type solid)) (layer "Edge.Cuts"))
+  (gr_line (start 110.1 59.9) (end 75.1 59.9)
+    (stroke (width 0.1) (type solid)) (layer "Edge.Cuts"))
+  (gr_line (start 183.3 82.4) (end 184.3 82.4)
+    (stroke (width 0.1) (type solid)) (layer "Edge.Cuts"))
+  (gr_line (start 135.1 82.75) (end 135.1 83.75)
+    (stroke (width 0.1) (type solid)) (layer "Edge.Cuts"))
+  (gr_circle (center 115.9 94.85) (end 117.85 94.85)
+    (stroke (width 0.1) (type solid)) (fill none) (layer "Edge.Cuts"))
+  (gr_line (start 173.3 98.1) (end 172.3 98.1)
+    (stroke (width 0.1) (type solid)) (layer "Edge.Cuts"))
+  (gr_circle (center 175.3 70.05) (end 177.25 70.05)
+    (stroke (width 0.1) (type solid)) (fill none) (layer "Edge.Cuts"))
+  (gr_circle (center 180.3 70.05) (end 181.45 70.05)
+    (stroke (width 0.1) (type solid)) (fill none) (layer "Edge.Cuts"))
+  (gr_line (start 173.3 98.1) (end 173.3 97.1)
+    (stroke (width 0.1) (type solid)) (layer "Edge.Cuts"))
+  (gr_rect (start 110.1 59.9) (end 198.3 99.7)
+    (stroke (width 0.1) (type solid)) (fill none) (layer "Edge.Cuts"))
+  (gr_line (start 135.1 82.7) (end 134.1 82.7)
+    (stroke (width 0.1) (type solid)) (layer "Edge.Cuts"))
+  (gr_line (start 135.1 82.7) (end 135.1 81.7)
+    (stroke (width 0.1) (type solid)) (layer "Edge.Cuts"))
+  (gr_line (start 135.1 82.7) (end 136.1 82.7)
+    (stroke (width 0.1) (type solid)) (layer "Edge.Cuts"))
+  (gr_line (start 110.1 99.7) (end 75.1 99.7)
+    (stroke (width 0.1) (type solid)) (layer "Edge.Cuts"))
+  (gr_line (start 183.3 82.4) (end 182.3 82.4)
+    (stroke (width 0.1) (type solid)) (layer "Edge.Cuts"))
   (gr_text "Rotary switch" (at 135.2 85.15) (layer "User.1")
     (effects (font (size 1 1) (thickness 0.15)))
@@
     (effects (font (size 1 1) (thickness 0.15)))
   )
+  (segment (start 88.51 145.42) (end 92.691974 149.601974) (width 0.25) (layer "F.Cu") (net 0))
+  (segment (start 104.385 147.325) (end 105.02 146.69) (width 0.25) (layer "F.Cu") (net 0))
+  (segment (start 94.86 150.5) (end 96.13 150.5) (width 0.25) (layer "F.Cu") (net 0))
+  (segment (start 98.298026 149.601974) (end 110.1 137.8) (width 0.25) (layer "F.Cu") (net 0))
+  (segment (start 104.385 147.696975) (end 104.385 147.325) (width 0.25) (layer "F.Cu") (net 0))
+  (segment (start 116.45 150.5) (end 107.56 150.5) (width 0.25) (layer "F.Cu") (net 0))
+  (segment (start 105.02 146.69) (end 104.861366 146.848634) (width 0.25) (layer "F.Cu") (net 0))
+  (segment (start 105.391975 149.601974) (end 105.02 149.23) (width 0.25) (layer "F.Cu") (net 0))
+  (segment (start 105.02 146.69) (end 113.91 137.8) (width 0.25) (layer "F.Cu") (net 0))
+  (via (at 88.51 145.42) (size 2) (drill 0.8) (layers "F.Cu" "B.Cu") (net 0))
+  (via (at 116.45 150.5) (size 2) (drill 0.8) (layers "F.Cu" "B.Cu") (net 0))
+  (arc (start 92.691974 149.601974) (mid 93.686672 150.266611) (end 94.86 150.5) (width 0.25) (layer "F.Cu") (net 0))
+  (arc (start 96.13 150.5) (mid 97.303328 150.266611) (end 98.298026 149.601974) (width 0.25) (layer "F.Cu") (net 0))
+  (arc (start 107.56 150.5) (mid 106.386673 150.266611) (end 105.391975 149.601974) (width 0.25) (layer "F.Cu") (net 0))
+  (arc (start 105.02 149.23) (mid 104.550032 148.526643) (end 104.385 147.696975) (width 0.25) (layer "F.Cu") (net 0))
+  (arc (start 104.861366 146.848634) (mid 104.520662 147.358532) (end 104.401023 147.96) (width 0.25) (layer "F.Cu") (net 0))
+  (segment (start 88.51 145.42) (end 110.1 145.42) (width 0.25) (layer "B.Cu") (net 0))
+  (segment (start 112.268025 146.318026) (end 112.64 146.69) (width 0.25) (layer "B.Cu") (net 0))
+  (segment (start 112.64 146.69) (end 116.45 150.5) (width 0.25) (layer "B.Cu") (net 0))
+  (arc (start 110.1 145.42) (mid 111.273327 145.653389) (end 112.268025 146.318026) (width 0.25) (layer "B.Cu") (net 0))
 )
