File: hw/ikea-fornuftig/ikea-fornuftig.kicad_sch (KiCad schematic)
At the start: 0 parts

Commit message: Updated title block of schematic file
Other:
- title: (none) -> IKEA FÖRNUFTIG Smart PCB
Changed lines of the file:
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@@
 (kicad_sch (version 20211123) (generator eeschema)
   (paper "A4")
+  (title_block
+    (title "IKEA FÖRNUFTIG Smart PCB")
+    (date "2023-01-07")
+    (comment 1 "https://jonas.lorander.com/")
+    (comment 2 "jonas@lorander.com")
+  )
   (sheet_instances
     (path "/" (page "1"))

Commit message: Description of motor interface added
Other:
- note added: "1. CLK controlls the speed of the fan a. Signal is 5V b. Speed 1: 100 kHz c. Speed 2: 220 kHz d. Speed 3: 300 kHz 2. FG is feedback from the fan a. Frevens is normally the same as CLK b. When filter is getting full fan will have more difficult to push the air and the freuency will increase on this PIN"
Changed lines of the file:
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@@
   (title_block
     (title "IKEA FÖRNUFTIG Smart PCB")
-    (date "2023-01-07")
+    (date "${DATE}")
     (comment 1 "https://jonas.lorander.com/")
     (comment 2 "jonas@lorander.com")
   )
+  (text "1. CLK controlls the speed of the fan\n  a. Signal is 5V\n  b. Speed 1: 100 kHz\n  c. Speed 2: 220 kHz\n  d. Speed 3: 300 kHz\n\n2. FG is feedback from the fan\n  a. Frevens is normally the same as CLK\n  b. When filter is getting full fan will have more difficult to push the air and the freuency will increase on this PIN"
+    (at 16.51 34.29 0)
+    (effects (font (size 1.27 1.27)) (justify left bottom))
+  )
   (sheet_instances
